File: hardware/kicad/loopy_pi_main.kicad_pcb (KiCad board)
At the start: 2 copper layers, 96 x 98 mm, 54 parts, among them J1 RPi_GPIO_HAT, J10 TRACK4, J11 CLEAR, J12 BANK, J13 RING, J14 IND, J17 I2C, J18 PWR, J19 5VA, J2 9V, J3 RECPLAY, J4 STOP, J5 UNDO, J6 MODE, J7 TRACK1, J8 TRACK2, J9 TRACK3, Q1 IRF9540N, U1 BUCK 5V, U2 LVL SHIFT

Commit message: feat(hardware): show the Pi 4 + standoffs in loopy_pi_main's own 3D viewer
Attach the Raspberry Pi 4 and four standoffs to loopy_pi_main.kicad_pcb as
board-only 3D models (kicad/pi_mating_model.py): no pads/silk/courtyard,
excluded from BOM/position/netlist, references hidden. Opening the board and
pressing Alt-3 now shows the mounted stack, with zero effect on Gerbers, drill
or DRC (geometry verified byte-identical; DRC still 0/0).

Pi model referenced via ${KIPRJMOD}/_models/RPi4.step (downloaded on demand by
pi_assemble.py, gitignored); standoffs from KiCad's bundled Wurth library via
${KICAD10_3DMODEL_DIR}.

Co-Authored-By: Claude Opus 4.8 <noreply@anthropic.com>
Parts:
- added PI4: , , F.Cu at (78.0, 60.0)
- added SO1: , , F.Cu at (49.0, 37.0)
- added SO2: , , F.Cu at (107.0, 37.0)
- added SO3: , , F.Cu at (49.0, 86.0)
- added SO4: , , F.Cu at (107.0, 86.0)
