File: hardware/kicad/loopy_pi_main.kicad_pcb (KiCad board)
At the start: 2 copper layers, 96 x 98 mm, 59 parts, among them J1 RPi_GPIO_HAT, J10 TRACK4, J11 CLEAR, J12 BANK, J13 RING, J14 IND, J17 I2C, J18 PWR, J19 5VA, J2 9V, J3 RECPLAY, J4 STOP, J5 UNDO, J6 MODE, J7 TRACK1, J8 TRACK2, J9 TRACK3, Q1 IRF9540N, U1 BUCK 5V, U2 LVL SHIFT

Commit message: feat(hardware): ribbon-connected Pi board + buck module + downloaded 3D model
Rework the Pi main board so it no longer stacks on the Pi and drops the
discrete switching supply:

- J1: 2x20 female stacking socket -> 2x20 male boxed IDC header + 40-pin
  ribbon to the Pi's GPIO. The board sits separately, so the Pi's tall
  USB/Ethernet jacks no longer foul it. Pinout stays 1:1 through the ribbon.
- Power: replace the LM2596 + catch diode + 33uH inductor with a 3-pin
  7805-compatible buck MODULE (Recom R-78H5.0 drop-in; Pololu D36V28F5 for
  full 3A Pi headroom). Synchronous, >90% efficient, runs cool -- no heatsink.
- Re-route loopy_pi_main.kicad_pcb to match the new J1 + buck footprints.

3D assembly tooling:
- Stop committing the 17 MB RaspberryPi4_ModelB.step (+ NOTICE). pi_assemble.py
  now downloads the Pi 4 model on first run into _models/ (gitignored) and adds
  Wurth standoffs from KiCad's bundled library.
- Drop pi_mating_model.py; document the render-only assembly flow in the design
  doc.

Co-Authored-By: Claude Opus 4.8 <noreply@anthropic.com>
Parts:
- removed PI4, SO1, SO2, SO3, SO4: , 
- H1, H2, H3, H4: value MountingHole_2.7mm_M2.5 -> MountingHole_3.2mm_M3; footprint MountingHole_2.7mm_M2.5 -> MountingHole_3.2mm_M3
- J1: value RPi_GPIO_HAT -> RPi_GPIO_Ribbon; footprint PinSocket_2x20_P2.54mm_Vertical -> IDC-Header_2x20_P2.54mm_Vertical; moved to F.Cu
- moved H4 40.9 mm to (122.0, 124.0)
- moved H3 37.8 mm to (36.0, 121.5)
- moved H2 15.3 mm to (122.0, 34.0)
- moved H1 13.5 mm to (35.5, 36.0)
- turned J1 to -90 degrees
